File: out/board.kicad_pcb (KiCad board)
At the start: 2 copper layers, 56 parts, among them U1 STM32F103C8T6

Commit message: krystal-radio: finish SDR build, YOLO ML pipeline, EMC tests, direction finding, page report, agent prompts
Parts:
- removed the C_AF_I at (17.0, -31.5)
- removed the C_AF_Q at (31.7, -39.0)
- removed the C_IN at (46.9, 4.32)
- removed the C_LO at (46.4, -1.48)
- removed the C_OPI at (17.0, -38.5)
- removed the C_OPQ at (44.7, -26.0)
- removed the C_QWC at (43.8, -8.83)
- removed the J_ANT at (0.00, 0.00)
- removed the L_MIX at (13.9, -20.1)
- removed the R_AF_I at (10.8, -44.2)
- removed the R_AF_Q at (4.62, -41.1)
- removed the R_BS at (48.8, -44.6)
- removed the R_LO at (3.79, -46.8)
- removed the R_OPI at (17.0, -44.2)
- removed the R_OPQ at (44.8, -33.2)
- removed the R_QWC at (44.7, -38.9)
- removed the R_TERM at (38.9, -20.2)
- removed the TP_ADC_I at (-0.83, -28.5)
- removed the TP_ADC_Q at (27.3, -1.55)
- removed the TP_ANT at (27.3, 4.25)
- removed the TP_FIL at (24.2, -26.1)
- removed the TP_LNA1_D at (12.4, -25.8)
- removed the TP_LNA2_D at (24.3, -20.3)
- removed the U_LDO at (13.6, -11.7)
- added C_AF_I: 100p, tscircuit:100p, F.Cu at (65.4, 84.3)
- added C_AF_Q: 100p, tscircuit:100p, F.Cu at (72.8, 84.3)
- added C_IN: 100p, tscircuit:100p, F.Cu at (109.8, 84.3)
- added C_LO: 100p, tscircuit:100p, F.Cu at (65.4, 78.4)
- added C_OPI: 100p, tscircuit:100p, F.Cu at (117.2, 78.4)
- added C_OPQ: 100p, tscircuit:100p, F.Cu at (124.6, 78.4)
- added C_QWC: 100p, tscircuit:100p, F.Cu at (72.8, 72.4)
- added J_ANT: SMA_EDGE, tscircuit:SMA_EDGE, F.Cu at (105.7, 126.6)
- added J_PWR: 5V_IN, tscircuit:5V_IN, F.Cu at (71.4, 132.3)
- added J_USB: USB_CDC, tscircuit:USB_CDC, F.Cu at (90.9, 132.3)
- added L_MIX: 600R@100MHz, tscircuit:600R_100MHz, F.Cu at (131.8, 66.3)
- added R_AF_I: 10k, tscircuit:10k, F.Cu at (80.2, 72.4)
- added R_AF_Q: 10k, tscircuit:10k, F.Cu at (87.5, 72.4)
- added R_BS: 1k, tscircuit:1k, F.Cu at (94.9, 72.4)
- added R_LO: 50, tscircuit:50, F.Cu at (131.7, 72.4)
- added R_OPI: 10k, tscircuit:10k, F.Cu at (65.4, 66.4)
- added R_OPQ: 10k, tscircuit:10k, F.Cu at (72.7, 66.4)
- added R_QWC: 1k, tscircuit:1k, F.Cu at (80.1, 66.4)
- added R_TERM: 50, tscircuit:50, F.Cu at (102.2, 66.4)
- added TP_ADC_I: TESTPOINT, tscircuit:TESTPOINT, F.Cu at (108.9, 106.0)
- added TP_ADC_Q: TESTPOINT, tscircuit:TESTPOINT, F.Cu at (117.9, 106.0)
- added TP_ANT: TESTPOINT, tscircuit:TESTPOINT, F.Cu at (126.9, 106.0)
- added TP_FIL: TESTPOINT, tscircuit:TESTPOINT, F.Cu at (66.2, 94.8)
- added TP_LNA1_D: TESTPOINT, tscircuit:TESTPOINT, F.Cu at (75.2, 94.8)
- added TP_LNA2_D: TESTPOINT, tscircuit:TESTPOINT, F.Cu at (84.2, 94.8)
- added U_LDO: AMS1117-3.3, tscircuit:AMS1117-3_3, F.Cu at (68.1, 107.1)
- added X_QWC1: LPJ-1, tscircuit:LPJ-1, F.Cu at (78.0, 110.4)
- added Y1: 8MHz, tscircuit:8MHz, F.Cu at (92.8, 94.1)
- C_ANA1: footprint Capacitor_SMD:C_0805_2012Metric -> tscircuit:10u
- C_ANA2, C_LDO2, C_MCU1, C_MCU2, C_MIX3: footprint Capacitor_SMD:C_0805_2012Metric -> tscircuit:100n
- C_BS1, C_LNA1, C_MIX1, C_MIX2: footprint Capacitor_SMD:C_0805_2012Metric -> tscircuit:100p
- C_BS2: footprint Capacitor_SMD:C_0805_2012Metric -> tscircuit:10p
- C_LDO1: footprint Capacitor_SMD:C_0805_2012Metric -> tscircuit:100u
- C_MCU3: footprint Capacitor_SMD:C_0805_2012Metric -> tscircuit:4u7
- C_OSC1, C_OSC2: footprint Capacitor_SMD:C_0805_2012Metric -> tscircuit:22p
- FB1: footprint Inductor_SMD:L_0805_2012Metric -> tscircuit:600R_100MHz
- L_BS1: footprint Inductor_SMD:L_1210_3225Metric -> tscircuit:100u
- L_LNA1, L_LNA2: footprint Inductor_SMD:L_1210_3225Metric -> tscircuit:18u
- Q_LNA1, Q_LNA2: footprint Package_TO_SOT_SMD:SOT-23 -> tscircuit:2N7002
- R_G1, R_G2: footprint Resistor_SMD:R_0805_2012Metric -> tscircuit:10k
- R_G3: footprint Resistor_SMD:R_0805_2012Metric -> tscircuit:4k7
- R_G4: footprint Resistor_SMD:R_0805_2012Metric -> tscircuit:2k2
- R_S1, R_S2: footprint Resistor_SMD:R_0805_2012Metric -> tscircuit:1k
- R_USB1, R_USB2: footprint Resistor_SMD:R_0805_2012Metric -> tscircuit:22
- U1: footprint Package_QFP:LQFP-48_7x7mm_P0.5mm -> tscircuit:STM32F103C8T6
- U_MIX1: footprint Package_SO:SOIC-8_3.9x4.9mm_P1.27mm -> tscircuit:LT5560
- U_OP1: footprint Package_SO:SOIC-8_3.9x4.9mm_P1.27mm -> tscircuit:OPA2134
- moved U1 189.1 mm to (129.4, 126.2)
- moved L_LNA2 176.1 mm to (134.0, 93.9)
- moved C_OSC1 174.9 mm to (132.0, 78.4)
- moved L_BS1 171.1 mm to (116.9, 93.9)
- moved R_G1 158.1 mm to (102.3, 72.4)
- moved C_LNA1 154.7 mm to (132.0, 84.3)
- moved C_MIX1 153.0 mm to (95.0, 78.4)
- moved FB1 152.3 mm to (124.3, 66.3)
- moved C_BS1 146.7 mm to (95.0, 84.3)
- moved R_G3 145.3 mm to (117.0, 72.4)
- moved R_G4 141.9 mm to (124.3, 72.4)
- moved C_LDO1 141.4 mm to (117.2, 84.3)
- moved C_ANA1 140.9 mm to (80.2, 84.3)
- moved C_LDO2 139.9 mm to (124.6, 84.3)
- moved Q_LNA1 139.1 mm to (100.8, 94.0)
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Connections:
- net USB_D+ renamed USB_DP
- net USB_D- renamed USB_D_
- C_ANA1 pad 1: +3V3_ANA -> (no net)
- C_ANA1 pad 2: GND -> (no net)
- C_ANA2 pad 1: +3V3_ANA -> (no net)
- C_ANA2 pad 2: GND -> (no net)
- C_BS2 pad 2: GND -> (no net)
- C_LDO1 pad 1: +3V3 -> (no net)
- C_LDO1 pad 2: GND -> (no net)
- C_LDO2 pad 1: +3V3 -> (no net)
- C_LDO2 pad 2: GND -> (no net)
- C_LNA1 pad 2: GND -> (no net)
- C_MCU1 pad 1: +3V3 -> (no net)
- C_MCU1 pad 2: GND -> (no net)
- C_MCU2 pad 1: +3V3 -> (no net)
- C_MCU2 pad 2: GND -> (no net)
- C_MCU3 pad 1: +3V3 -> (no net)
- C_MCU3 pad 2: GND -> (no net)
- C_MIX2 pad 1: GND -> (no net)
- C_MIX3 pad 2: GND -> (no net)
- C_OSC1 pad 2: GND -> (no net)
- C_OSC2 pad 2: GND -> (no net)
- FB1 pad 1: +3V3 -> (no net)
- FB1 pad 2: +3V3_ANA -> (no net)
- L_LNA1 pad 1: +3V3 -> (no net)
- L_LNA2 pad 1: +3V3_ANA -> (no net)
- R_G1 pad 1: +3V3 -> (no net)
- R_G2 pad 2: GND -> (no net)
- R_G3 pad 1: +3V3 -> (no net)
- R_G4 pad 2: GND -> (no net)
- R_S1 pad 2: GND -> (no net)
- R_S2 pad 2: GND -> (no net)
- R_USB1 pad 2: USB_D+_R -> (no net)
- R_USB2 pad 2: USB_D-_R -> (no net)
- U1 pad 1: +3V3 -> (no net)
- U1 pad 2: GND -> (no net)
- U1 pad 3: +3V3 -> (no net)
- U1 pad 9: CTRL -> (no net)
- U_OP1 pad 7: +3V3_ANA -> (no net)
- U_OP1 pad 8: GND -> (no net)
Routing:
- net USB_DP: track 0.00 -> 105.4 mm, vias 0 -> 4
- net USB_D_: track 0.00 -> 104.9 mm, vias 0 -> 6
- net LO: track 0.00 -> 101.0 mm, vias 0 -> 10
- net ADC_I_F: track 0.00 -> 98.9 mm, vias 0 -> 8
- net ADC_Q_F: track 0.00 -> 95.9 mm, vias 0 -> 8
- net RF_IN: track 0.00 -> 87.7 mm, vias 0 -> 8
- net ADC_Q: track 0.00 -> 87.1 mm, vias 0 -> 10
- net LNA1_D: track 0.00 -> 79.8 mm, vias 0 -> 14
- net ADC_I: track 0.00 -> 78.1 mm, vias 0 -> 9
- net LNA2_G: track 0.00 -> 74.8 mm, vias 0 -> 9
- net FIL_OUT: track 0.00 -> 74.5 mm, vias 0 -> 8
- net LNA1_S: track 0.00 -> 72.0 mm, vias 0 -> 9
- net VCC_MIX: track 0.00 -> 67.6 mm, vias 0 -> 9
- net MIX_Q1: track 0.00 -> 67.2 mm, vias 0 -> 4
- net LNA2_D: track 0.00 -> 66.3 mm, vias 0 -> 6
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- added copper zone on B.Cu, net GND
- added copper zone on In1.Cu, net GND
- added copper zone on In2.Cu, net P3V3
- added copper zone on F.Cu, net P3V3_ANA
Other:
- board outline added: 88.6 x 85.1 mm
- copper layers 2 -> 4
- board text added: "C_0805_2012Metric"
- board text added: "Crystal_SMD_3225-4Pin_3.2x2.5mm"
- board text added: "LQFP-48_7x7mm_P0.5mm"
- board text added: "L_0805_2012Metric"
- board text added: "L_1210_3225Metric"
- board text added: "PinHeader_1x04_P1.27mm_Vertical"
- board text added: "REF**"
- board text added: "R_0805_2012Metric"
- board text added: "SMA_Amphenol_132289_EdgeMount"
- board text added: "SOIC-8_3.9x4.9mm_P1.27mm"
- board text added: "SOT-223-3_TabPin2"
- board text added: "SOT-23"
- board text added: "TestPoint_Pad_D1.5mm"
- board text added: "USB_B_TE_5787834_Vertical"
